File: SCD41-D-R1_demo.kicad_pcb (KiCad board)
At the start: 2 copper layers, 43.8 x 40 mm, 18 parts, among them J1 USB_A, J3 Prog, U1 SCD41-D-R2, U2 AP2112K-3.3, U3 USBLC6-2SC6, U4 ESP32-WROOM-32

Commit message: programmer
Parts:
- added C9: 10u, Capacitor_SMD:C_0603_1608Metric, F.Cu at (191.0, 88.2)
- added Q1: BC846BS, Package_TO_SOT_SMD:SOT-363_SC-70-6, F.Cu at (196.9, 78.0)
- added R13: 1k, Resistor_SMD:R_0603_1608Metric, F.Cu at (193.8, 94.0)
- added R14: 10k, Resistor_SMD:R_0603_1608Metric, F.Cu at (196.8, 81.0)
- added R15: 10k, Resistor_SMD:R_0603_1608Metric, F.Cu at (197.2, 75.0)
- added U7: CP2102N-Axx-xQFN28, Package_DFN_QFN:QFN-28-1EP_5x5mm_P0.5mm_EP3.35x3.35mm, F.Cu at (195.0, 90.0)
- moved C2 3.90 mm to (183.0, 92.5)
- moved C3 3.90 mm to (183.3, 87.9)
- moved C4 3.90 mm to (187.5, 86.4)
- moved U2 3.90 mm to (187.0, 89.0)
- moved FB1 3.90 mm to (183.0, 91.0)
- moved U3 3.90 mm to (188.1, 92.9)
Connections:
- net D0 renamed BT

Commit message: usb-c
Parts:
- removed J1: USB_A, Connector_USB:USB_Mini-B_Wuerth_65100516121_Horizontal
- added J4: USB_C_Receptacle, Connector_USB:USB_C_Receptacle_HRO_TYPE-C-31-M-12, F.Cu at (187.0, 101.4)
- added R1: 5k1, Resistor_SMD:R_0805_2012Metric, F.Cu at (180.0, 102.0)
- added R5: 5k1, Resistor_SMD:R_0805_2012Metric, F.Cu at (194.0, 100.9)
Connections:
- U3 pad 1: Net-(J1-D+) -> D+
- U3 pad 3: Net-(J1-D-) -> D-

Commit message: layout
Parts:
- moved R14 0.56 mm to (197.1, 80.5)
Connections:
- J4 pad A4: +5V -> VIN
- J4 pad A9: +5V -> VIN
- J4 pad B4: +5V -> VIN
- J4 pad B9: +5V -> VIN
- R16 pad 1: +3V3 -> +3.3V
- R17 pad 1: +3V3 -> +3.3V
- U3 pad 5: +5V -> VIN
- U7 pad 8: +5V -> VIN
Routing:
- net SCL: track 0.00 -> 40.9 mm, vias 0 -> 2
- net GND: track 0.00 -> 36.4 mm, vias 0 -> 23
- net SDA: track 0.00 -> 31.5 mm
- net EN: track 0.00 -> 30.3 mm, vias 0 -> 2
- net TX: track 0.00 -> 26.9 mm, vias 0 -> 2
- net VIN: track 0.00 -> 25.9 mm, vias 0 -> 2
- net RX: track 0.00 -> 22.9 mm, vias 0 -> 2
- net BT: track 0.00 -> 20.1 mm
- net +3.3V: track 0.00 -> 14.9 mm, vias 0 -> 15
- net Net-(Q1A-E1): track 0.00 -> 14.0 mm, vias 0 -> 2
- net Net-(Q1B-E2): track 0.00 -> 11.7 mm
- net Net-(J4-CC1): track 0.00 -> 8.45 mm
- net Net-(U2-EN): track 0.00 -> 7.59 mm
- net D-: track 0.00 -> 7.42 mm
- net Net-(J4-CC2): track 0.00 -> 7.06 mm
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- added copper zone on In2.Cu, net +3.3V
- added copper zone on In1.Cu, net GND
Other:
- board size 43.8 x 40 mm -> 41.1 x 40 mm
- copper layers 2 -> 4
